File: transponder/transponder.sch (KiCad schematic (older format))
At the start: 6 parts, among them IC1 ATTINY45-S, P1 POWER_CONN, P2 CONN_01X05

Commit message: transponder: Rewire LED
Connections:
- net PROG_MISO: now also R1.1
- net at IC1.2 (PB3(XTAL1/CLKI/OC1B/ADC3/PCINT3)): no longer R1.1
- no-connect marks 1 -> 2
Changed lines of the file:
@@
 	4900 3300 5350 3300
 Wire Wire Line
-	5350 3400 4900 3400
+	4450 3400 5350 3400
 Wire Wire Line
 	5350 3500 4900 3500
 Wire Wire Line
 	5350 3800 4900 3800
-Wire Wire Line
-	5350 3600 4450 3600
 Wire Wire Line
 	4450 3900 4450 3950
@@
 	-1   0    0    1
 $EndComp
+Wire Wire Line
+	4450 3600 4450 3400
+NoConn ~ 5350 3600
 $EndSCHEMATC
